File: pcb_kicad/barehub.kicad_sch (KiCad schematic)
At the start: 32 parts, among them J2 USB_A, J3 USB_A, J4 USB_A, J5 USB_A, J6 USB_C_Receptacle_USB2.0_16P, U1 FE1.1s, U2 SMF05CT1G, U3 SMF05CT1G, U4 SMF05CT1G, U5 SMF05CT1G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

Commit message: chore: add BOM
Other:
- note added: "22/2/2026"
- note added: "BAREHUB - BLUEPRINT"
- note added: "DECOUPLING - CAPS"
- note added: "DOWNSTREAM - USBA"
- note added: "FE1.1S - IC"
- note added: "UPSTREAM - USBC"
- moved on the sheet: C11, C12, C2, C3, D1, F5, J6, R1, R2, R4, R5, R6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
